File: SpexPressureSensor.sch (KiCad schematic (older format))
At the start: 28 parts, among them P1 CONN_6, P2 NICHROME, P3 TC2030-CTX, Q1 IRLL3303PbF, U1 ST1480ABDR, U2 TPS769XX, U3 MKL03ZxxVFG4, U4 BMP180, U7 LT6105

Commit message: Commiting the rest of teh files
Parts:
- removed U4: BMP180, BMP180:LGA7-1.5-3.8X3.6MM, symbol BMP180
- added U4: BME280, bme280:LGA-8, symbol BME280
Connections:
- wire segments 116 -> 119
Changed lines of the file:
@@
 LIBS:Tag-Connect
 LIBS:lt6105
+LIBS:bme280
 LIBS:SpexPressureSensor-cache
 EELAYER 25 0
@@
 $EndComp
 $Comp
-L BMP180 U4
-U 1 1 5647E74D
-P 8350 3950
-F 0 "U4" H 8700 4050 50  0000 C CNN
-F 1 "BMP180" H 8700 4150 50  0000 C CNN
-F 2 "BMP180:LGA7-1.5-3.8X3.6MM" H 8350 3950 50  0001 C CNN
-F 3 "DOCUMENTATION" H 8350 3950 50  0001 C CNN
-	1    8350 3950
-	1    0    0    -1
-$EndComp
-$Comp
 L C-RESCUE-SpexPressureSensor C7
 U 1 1 5647E7A7
@@
 	8300 3400 8300 3300
 Wire Wire Line
-	8300 3300 9150 3300
+	7500 3300 9150 3300
 Wire Wire Line
 	8350 3300 8350 3250
@@
 Connection ~ 8400 3300
 Wire Wire Line
-	9150 4150 9150 4550
-Wire Wire Line
-	9150 4550 8300 4550
+	9150 4550 9150 4150
+Wire Wire Line
+	7500 4550 9150 4550
 Wire Wire Line
 	8300 4500 8300 4700
@@
 Text Notes 550  5200 0    60   ~ 0
 .2v per amp
+$Comp
+L BME280 U4
+U 1 1 570B033C
+P 8350 3950
+F 0 "U4" H 8928 3996 50  0000 L CNN
+F 1 "BME280" H 8928 3905 50  0000 L CNN
+F 2 "bme280:LGA-8" H 8350 3950 50  0001 C CNN
+F 3 "DOCUMENTATION" H 8350 3950 50  0001 C CNN
+	1    8350 3950
+	1    0    0    -1
+$EndComp
+Wire Wire Line
+	8200 4500 8200 4550
+Wire Wire Line
+	7500 3800 7500 3300
+Connection ~ 8300 3300
+Wire Wire Line
+	7500 4100 7500 4550
+Connection ~ 8200 4550
 $EndSCHEMATC

Commit message: Fixed some issues
Parts:
- U2: Manufacturer PN (none) -> NCP500SN33T1G
Changed lines of the file:
@@
 F 2 "Housings_SOT-23_SOT-143_TSOT-6:SOT-23-5" H 3200 1550 60  0001 C CNN
 F 3 "" H 3200 1550 60  0000 C CNN
+F 4 "NCP500SN33T1G" H 3200 1550 60  0001 C CNN "Manufacturer PN"
 	1    3200 1550
 	1    0    0    -1
